Commit message: fixed the physical placement of camera, need to adjust where the position of the images being output

File: car_ros/description/robot_camera.xacro (robot description, xacro)
@@ -5,21 +5,21 @@
             <update_rate>30.0</update_rate>
             <camera name="head">
-                <horizontal_fov>1.3962634</horizontal_fov>
+                <horizontal_fov>1.085595</horizontal_fov>
                 <image>
-                <width>800</width>
-                <height>800</height>
-                <format>R8G8B8</format>
+                    <width>3280</width>
+                    <height>2464</height>
+                    <format>R8G8B8</format>
                 </image>
                 <clip>
-                <near>0.02</near>
-                <far>300</far>
+                    <near>0.02</near>
+                    <far>300</far>
                 </clip>
                 <noise>
-                <type>gaussian</type>
-                <!-- Noise is sampled independently per pixel on each frame.
-                    That pixel's noise value is added to each of its color
-                    channels, which at that point lie in the range [0,1]. -->
-                <mean>0.0</mean>
-                <stddev>0.007</stddev>
+                    <type>gaussian</type>
+                    <!-- Noise is sampled independently per pixel on each frame.
+                        That pixel's noise value is added to each of its color
+                        channels, which at that point lie in the range [0,1]. -->
+                    <mean>0.0</mean>
+                    <stddev>0.007</stddev>
                 </noise>
             </camera>

File: car_ros/description/robot_core.xacro (robot description, xacro)
@@ -32,5 +32,5 @@
             <origin xyz="0.17 0 0.075"/>
             <geometry>
-                <box size="0.33 0.15 0.15"/>
+                <box size="0.3302 0.1524 0.15"/>
             </geometry>
             <material name="black"/>
@@ -163,6 +163,6 @@
     <!-- CAMERA LINK -->
     <joint name="camera_joint" type="fixed">
-        <axis xyz="0 1 0" />
-        <origin xyz="0.17 0 0.075" rpy="0 0 0"/>
+        <axis xyz="0 -0.0020 0.1016" />
+        <origin xyz="0 -0.0020 0.1016" rpy="0 0 0"/>
         <parent link="base_link"/>
         <child link="camera_link"/>
@@ -170,5 +170,5 @@
     <link name="camera_link">
         <collision>
-            <origin xyz="0.09 0.05 0" rpy="0 0 0"/>
+            <origin xyz="0 -0.0020 0.1016" rpy="0 0 0"/>
             <geometry>
                 <box size="${camera_link} ${camera_link} ${camera_link}"/>
@@ -176,5 +176,5 @@
         </collision>
         <visual>
-            <origin xyz="0.09 0.05 0" rpy="0 0 0"/>
+            <origin xyz="0.08 0 0.075" rpy="0 0 0"/>
             <geometry>
                 <box size="${camera_link} ${camera_link} ${camera_link}"/>
@@ -184,5 +184,5 @@
         <inertial>
             <mass value="1e-5" />
-            <origin xyz="0.09 0.05 0" rpy="0 0 0"/>
+            <origin xyz="0 -0.0020 0.1016" rpy="0 0 0"/>
             <inertia ixx="1e-6" ixy="0" ixz="0" iyy="1e-6" iyz="0" izz="1e-6" />
         </inertial>
