Commit message: camera is working and displays on rviz, just need to fix the positioning to make it more accurate to the model

File: car_ros/description/robot.urdf.xacro (robot description, xacro)
@@ -3,3 +3,4 @@
      <xacro:include filename="robot_core.xacro"/>
      <xacro:include filename="gazebo_control.xacro"/>
+     <xacro:include filename="robot_camera.xacro"/>
 </robot>

File: car_ros/description/robot_core.xacro (robot description, xacro)
@@ -2,4 +2,5 @@
 <robot xmlns:xacro="http://www.ros.org/wiki/xacro" >
     <xacro:include filename="inertial_macros.xacro"/>
+    <xacro:include filename="robot_camera.xacro"/>
     <material name="white">
         <color rgba="1 1 1 1" />
@@ -17,4 +18,5 @@
         <color rgba="1 0 0 1"/>
     </material>
+    <xacro:property name="camera_link" value="0.05" />
     <!-- BASE LINK -->
     <link name="base_link">
@@ -159,3 +161,33 @@
         <mu2 value="0.018"/>
     </gazebo>
+    <!-- CAMERA LINK -->
+    <joint name="camera_joint" type="fixed">
+        <axis xyz="0 1 0" />
+        <origin xyz="0.17 0 0.075" rpy="0 0 0"/>
+        <parent link="base_link"/>
+        <child link="camera_link"/>
+    </joint>
+    <link name="camera_link">
+        <collision>
+            <origin xyz="0.09 0.05 0" rpy="0 0 0"/>
+            <geometry>
+                <box size="${camera_link} ${camera_link} ${camera_link}"/>
+            </geometry>
+        </collision>
+        <visual>
+            <origin xyz="0.09 0.05 0" rpy="0 0 0"/>
+            <geometry>
+                <box size="${camera_link} ${camera_link} ${camera_link}"/>
+            </geometry>
+            <material name="red"/>
+        </visual>
+        <inertial>
+            <mass value="1e-5" />
+            <origin xyz="0.09 0.05 0" rpy="0 0 0"/>
+            <inertia ixx="1e-6" ixy="0" ixz="0" iyy="1e-6" iyz="0" izz="1e-6" />
+        </inertial>
+    </link>
+    <gazebo reference="camera_link">
+        <material>Gazebo/Red</material>
+    </gazebo>
 </robot>

Commit message: Car is updated, need to fix the lidar

File: car_ros/description/robot.urdf.xacro (robot description, xacro)
@@ -4,3 +4,4 @@
      <xacro:include filename="gazebo_control.xacro"/>
      <xacro:include filename="robot_camera.xacro"/>
+     <xacro:include filename="robot_lidar.xacro"/>
 </robot>

File: car_ros/description/robot_core.xacro (robot description, xacro)
@@ -3,4 +3,5 @@
     <xacro:include filename="inertial_macros.xacro"/>
     <xacro:include filename="robot_camera.xacro"/>
+    <xacro:include filename="robot_lidar.xacro"/>
     <material name="white">
         <color rgba="1 1 1 1" />
@@ -191,3 +192,33 @@
         <material>Gazebo/Red</material>
     </gazebo>
+    <!-- LIDAR LINK -->
+    <joint name="hokuyo_joint" type="fixed">
+        <axis xyz="0 1 0" />
+        <origin xyz="0 0 0.1143" rpy="0 0 0"/>
+        <parent link="base_link"/>
+        <child link="hokuyo_link"/>
+    </joint>
+    <!-- Hokuyo Laser -->
+    <link name="hokuyo_link">
+        <collision>
+            <origin xyz="0 0 0" rpy="0 0 0"/>
+            <geometry>
+                <box size="0.02 0.02 0.01"/>
+            </geometry>
+        </collision>
+        <visual>
+            <origin xyz="0 0 0" rpy="0 0 0"/>
+            <geometry>
+                <box size="0.02 0.02 0.01"/>
+            </geometry>
+        </visual>
+        <inertial>
+            <mass value="1e-5" />
+            <origin xyz="0 0 0" rpy="0 0 0"/>
+            <inertia ixx="1e-6" ixy="0" ixz="0" iyy="1e-6" iyz="0" izz="1e-6" />
+        </inertial>
+    </link>
+    <gazebo reference="hokuyo_link">
+        <material>Gazebo/Orange</material>
+    </gazebo>
 </robot>
