Commit message: able to turn, going to try to make it more smoother/easier to control

File: car_ros/description/robot_core.xacro (robot description, xacro)
@@ -2,4 +2,5 @@
 <robot xmlns:xacro="http://www.ros.org/wiki/xacro" >
     <xacro:include filename="inertial_macros.xacro"/>
+    <xacro:include filename = "summit_base.gazebo.xacro"/>
     <material name="white">
         <color rgba="1 1 1 1" />
@@ -32,5 +33,5 @@
                 <box size="0.33 0.15 0.15"/>
             </geometry>
-            <material name="white"/>
+            <material name="black"/>
         </visual>
         <collision>
@@ -43,7 +44,9 @@
             <origin xyz="0.17 0 0.075" rpy="0 0 0"/>
         </xacro:inertial_box>
+        <xacro:omni_steering>
+        </xacro:omni_steering>
     </link>
     <gazebo reference="chassis">
-        <material>Gazebo/White</material>
+        <material>Gazebo/Black</material>
     </gazebo>
     <!-- FRONT LEFT WHEEL LINK -->

Commit message: Issue: rviz2 shows wheels when the wheel's joint type is fixed, however, the wheels wont rotate in gazebo or in rviz2. WHen wheel's joint type is continuous the wheels rotate in gazebo, however, they dont show up in rviz2

File: car_ros/description/robot_core.xacro (robot description, xacro)
@@ -48,5 +48,5 @@
     </gazebo>
     <!-- FRONT LEFT WHEEL LINK -->
-    <joint name="front_left_wheel_joint" type="continuous">
+    <joint name="front_left_wheel_joint" type="fixed">
         <parent link="base_link"/>
         <child link="front_left_wheel"/>
@@ -76,5 +76,5 @@
     </gazebo>
     <!-- BACK LEFT WHEEL LINK -->
-    <joint name="back_left_wheel_joint" type="continuous">
+    <joint name="back_left_wheel_joint" type="fixed">
         <parent link="base_link"/>
         <child link="back_left_wheel"/>
@@ -104,5 +104,5 @@
     </gazebo>
     <!-- FRONT RIGHT WHEEL LINK -->
-    <joint name="front_right_wheel_joint" type="continuous">
+    <joint name="front_right_wheel_joint" type="fixed">
         <parent link="base_link"/>
         <child link="front_right_wheel"/>
@@ -132,5 +132,5 @@
     </gazebo>
     <!-- BACK RIGHT WHEEL LINK -->
-    <joint name="back_right_wheel_joint" type="continuous">
+    <joint name="back_right_wheel_joint" type="fixed">
         <parent link="base_link"/>
         <child link="back_right_wheel"/>

Commit message: fix

File: car_ros/description/robot_core.xacro (robot description, xacro)
@@ -115,5 +115,5 @@
                 <cylinder radius="0.04" length="0.03"/>
             </geometry>
-            <material name="blue"/>hjnbm
+            <material name="blue"/>
         </visual>
         <collision>

Commit message: added camera and updated wheels

File: car_ros/description/robot_core.xacro (robot description, xacro)
@@ -59,5 +59,5 @@
         <visual>
             <geometry>
-                <cylinder radius="0.04" length="0.03"/>
+                <cylinder radius="0.032" length="0.03"/>
             </geometry>
             <material name="blue"/>
@@ -65,5 +65,5 @@
         <collision>
             <geometry>
-                <cylinder radius="0.04" length="0.03"/>
+                <cylinder radius="0.032" length="0.03"/>
             </geometry>
         </collision>
@@ -87,5 +87,5 @@
         <visual>
             <geometry>
-                <cylinder radius="0.04" length="0.03"/>
+                <cylinder radius="0.032" length="0.03"/>
             </geometry>
             <material name="blue"/>
@@ -93,5 +93,5 @@
         <collision>
             <geometry>
-                <cylinder radius="0.04" length="0.03"/>
+                <cylinder radius="0.032" length="0.03"/>
             </geometry>
         </collision>
@@ -115,5 +115,5 @@
         <visual>
             <geometry>
-                <cylinder radius="0.04" length="0.03"/>
+                <cylinder radius="0.032" length="0.03"/>
             </geometry>
             <material name="blue"/>
@@ -121,5 +121,5 @@
         <collision>
             <geometry>
-                <cylinder radius="0.04" length="0.03"/>
+                <cylinder radius="0.032" length="0.03"/>
             </geometry>
         </collision>
@@ -143,5 +143,5 @@
         <visual>
             <geometry>
-                <cylinder radius="0.04" length="0.03"/>
+                <cylinder radius="0.032" length="0.03"/>
             </geometry>
             <material name="blue"/>hjnbm
@@ -149,5 +149,5 @@
         <collision>
             <geometry>
-                <cylinder radius="0.04" length="0.03"/>
+                <cylinder radius="0.032" length="0.03"/>
             </geometry>
         </collision>

Commit message: fixed positioning of the camera and its specs to align with the model and raspberry pi camera v2 respectively

File: car_ros/description/robot_core.xacro (robot description, xacro)
@@ -30,5 +30,5 @@
     <link name="chassis">
         <visual>
-            <origin xyz="0.17 0 0.075"/>
+            <origin xyz="0.1778 0 0.075"/>
             <geometry>
                 <box size="0.3302 0.1524 0.15"/>
@@ -37,5 +37,5 @@
         </visual>
         <collision>
-            <origin xyz="0.17 0 0.075"/>
+            <origin xyz="0.1778 0 0.075"/>
             <geometry>
                 <box size="0.3302 0.1524 0.15"/>
@@ -43,5 +43,5 @@
         </collision>
         <xacro:inertial_box mass="0.5" x="0.33" y="0.15" z="0.15">
-            <origin xyz="0.17 0 0.075" rpy="0 0 0"/>
+            <origin xyz="0.1778 0 0.075" rpy="0 0 0"/>
         </xacro:inertial_box>
     </link>
@@ -137,5 +137,5 @@
         <parent link="base_link"/>
         <child link="back_right_wheel"/>
-        <origin xyz="0 -0.091 0" rpy="${pi/2} 0 0" />
+        <origin xyz="-0.0128 -0.091 0" rpy="${pi/2} 0 0" />
         <axis xyz="0 0 -1"/>
     </joint>
@@ -163,6 +163,6 @@
     <!-- CAMERA LINK -->
     <joint name="camera_joint" type="fixed">
-        <axis xyz="0 -0.0020 0.1016" />
-        <origin xyz="0 -0.0020 0.1016" rpy="0 0 0"/>
+        <axis xyz="0 0 0" />
+        <origin xyz="0.08 -0.0020 0.2286" rpy="0 0 0"/>
         <parent link="base_link"/>
         <child link="camera_link"/>
@@ -170,5 +170,5 @@
     <link name="camera_link">
         <collision>
-            <origin xyz="0 -0.0020 0.1016" rpy="0 0 0"/>
+            <origin xyz="0.08 -0.0020 0.2286" rpy="0 0 0"/>
             <geometry>
                 <box size="${camera_link} ${camera_link} ${camera_link}"/>
@@ -176,5 +176,5 @@
         </collision>
         <visual>
-            <origin xyz="0.08 0 0.075" rpy="0 0 0"/>
+            <origin xyz="0 0 0" rpy="0 0 0"/>
             <geometry>
                 <box size="${camera_link} ${camera_link} ${camera_link}"/>
@@ -184,5 +184,5 @@
         <inertial>
             <mass value="1e-5" />
-            <origin xyz="0 -0.0020 0.1016" rpy="0 0 0"/>
+            <origin xyz="0.08 -0.0020 0.2286" rpy="0 0 0"/>
             <inertia ixx="1e-6" ixy="0" ixz="0" iyy="1e-6" iyz="0" izz="1e-6" />
         </inertial>

Commit message: implemented the lidar, need to tweak it to follow the parameters of our model

File: car_ros/description/robot_core.xacro (robot description, xacro)
@@ -2,6 +2,4 @@
 <robot xmlns:xacro="http://www.ros.org/wiki/xacro" >
     <xacro:include filename="inertial_macros.xacro"/>
-    <xacro:include filename="robot_camera.xacro"/>
-    <xacro:include filename="robot_lidar.xacro"/>
     <material name="white">
         <color rgba="1 1 1 1" />
@@ -192,33 +190,3 @@
         <material>Gazebo/Red</material>
     </gazebo>
-    <!-- LIDAR LINK -->
-    <joint name="hokuyo_joint" type="fixed">
-        <axis xyz="0 1 0" />
-        <origin xyz="0 0 0.1143" rpy="0 0 0"/>
-        <parent link="base_link"/>
-        <child link="hokuyo_link"/>
-    </joint>
-    <!-- Hokuyo Laser -->
-    <link name="hokuyo_link">
-        <collision>
-            <origin xyz="0 0 0" rpy="0 0 0"/>
-            <geometry>
-                <box size="0.02 0.02 0.01"/>
-            </geometry>
-        </collision>
-        <visual>
-            <origin xyz="0 0 0" rpy="0 0 0"/>
-            <geometry>
-                <box size="0.02 0.02 0.01"/>
-            </geometry>
-        </visual>
-        <inertial>
-            <mass value="1e-5" />
-            <origin xyz="0 0 0" rpy="0 0 0"/>
-            <inertia ixx="1e-6" ixy="0" ixz="0" iyy="1e-6" iyz="0" izz="1e-6" />
-        </inertial>
-    </link>
-    <gazebo reference="hokuyo_link">
-        <material>Gazebo/Orange</material>
-    </gazebo>
 </robot>

File: car_ros/description/robot_lidar.xacro (robot description, xacro)
@@ -1,38 +1,55 @@
 <?xml version="1.0"?>
-<robot xmlns:xacro="http://www.ros.org/wiki/xacro"  name="robot">
-  <gazebo reference="hokuyo_link">
-        <sensor type="gpu_ray" name="head_hokuyo_sensor">
-            <pose>0 0 0 0 0 0</pose>
+<robot xmlns:xacro="http://www.ros.org/wiki/xacro">
+    <joint name="laser_joint" type="fixed">
+        <parent link="chassis"/>
+        <child link="laser_frame"/>
+        <origin xyz = "0.08 0 0.1143" rpy="0 0 0"/>
+    </joint>
+    <link name = "laser_frame">
+        <visual>
+            <geometry>
+                <mesh filename="description/hokuyo.dae"/>
+            </geometry>
+        </visual>
+        <collision>
+            <origin xyz="0 0 0" rpy="0 0 0"/>
+            <geometry>
+                <box size="0.1 0.1 0.1"/>
+            </geometry>
+        </collision>
+        <inertial>
+            <mass value="1e-5" />
+            <origin xyz="0 0 0" rpy="0 0 0"/>
+            <inertia ixx="1e-6" ixy="0" ixz="0" iyy="1e-6" iyz="0" izz="1e-6" />
+        </inertial>
+    </link>
+    <gazebo reference="laser_frame">
+        <sensor name="laser" type="ray">
+            <pose> 0 0 0 0 0 0 </pose>
             <visualize>true</visualize>
-            <update_rate>40</update_rate>
+            <update_rate>10</update_rate>
             <ray>
                 <scan>
                     <horizontal>
-                        <samples>720</samples>
+                        <samples>360</samples>
                         <resolution>1</resolution>
-                        <min_angle>-1.570796</min_angle>
-                        <max_angle>1.570796</max_angle>
+                        <min_angle>-3.14</min_angle>
+                        <max_angle>3.14</max_angle>
                     </horizontal>
                 </scan>
                 <range>
-                    <min>0.10</min>
-                    <max>30.0</max>
+                    <min>0.3</min>
+                    <max>12</max>
                     <resolution>0.01</resolution>
                 </range>
-                <noise>
-                    <type>gaussian</type>
-                    <!-- Noise parameters based on published spec for Hokuyo laser
-                        achieving "+-30mm" accuracy at range < 10m.  A mean of 0.0m and
-                        stddev of 0.01m will put 99.7% of samples within 0.03m of the true
-                        reading. -->
-                    <mean>0.0</mean>
-                    <stddev>0.01</stddev>
-                </noise>
             </ray>
-            <plugin name="gazebo_ros_head_hokuyo_controller" filename="libgazebo_ros_gpu_laser.so">
-                <topicName>lidar_info</topicName>
-                <frameName>hokuyo_link</frameName>
+            <plugin name="laser_controller" filename="libgazebo_ros_ray_sensor.so">
+                <ros>
+                    <argument>~/out:=scan</argument>
+                </ros>
+                <output_type>sensor_msgs/LaserScan</output_type>
+                <frame_name>laser_frame</frame_name>
             </plugin>
         </sensor>
-  </gazebo>
+    </gazebo>
 </robot>

Commit message: able to rotate the lidar in RVIZ, but not in Gazebo

File: car_ros/description/robot_core.xacro (robot description, xacro)
@@ -190,3 +190,36 @@
         <material>Gazebo/Red</material>
     </gazebo>
+    <!-- ROTATING LINK -->
+    <joint name="rotate_joint" type="revolute">
+        <parent link="base_link"/>
+        <child link="rotate_link"/>
+        <origin xyz="-0.02 0 0.225" rpy="0 0 0"/>
+        <axis xyz="0 0 -1"/>
+        <limit lower="0" upper="${pi}" velocity="100" effort="100"/>
+    </joint>
+    <link name="rotate_link">
+        <visual>
+            <origin xyz="0 0 0" rpy="0 0 0"/>
+            <geometry>
+                <cylinder length="0.025" radius="0.025" />
+            </geometry>
+            <material name="orange" />
+        </visual>
+        <collision>
+            <origin xyz="0 0 0" rpy="-3.14159 0 0"/>
+            <geometry>
+                <cylinder length="0.001" radius="0.025" />
+            </geometry>
+        </collision>
+        <xacro:inertial_cylinder mass="0.01" length="0.001" radius="0.025">
+            <origin xyz="0 0 0" rpy="0 0 0"/>
+        </xacro:inertial_cylinder>
+    </link>
+    <gazebo>
+        <plugin name="gazebo_ros_joint_state_publisher"
+            filename="libgazebo_ros_joint_state_publisher.so">
+            <update_rate>40</update_rate>
+            <joint_name>rotate_link</joint_name>
+        </plugin>
+    </gazebo>
 </robot>

File: car_ros/description/robot_lidar.xacro (robot description, xacro)
@@ -2,12 +2,13 @@
 <robot xmlns:xacro="http://www.ros.org/wiki/xacro">
     <joint name="laser_joint" type="fixed">
-        <parent link="chassis"/>
+        <origin xyz = "0 0 0.025" rpy="0 0 0"/>
+        <parent link="rotate_link"/>
         <child link="laser_frame"/>
-        <origin xyz = "0.08 0 0.1143" rpy="0 0 0"/>
     </joint>
     <link name = "laser_frame">
         <visual>
+            <origin xyz = "0 0 0" rpy="0 0 0"/>
             <geometry>
-                <mesh filename="description/hokuyo.dae"/>
+                <box size="0.06 0.05 0.05" />
             </geometry>
         </visual>
@@ -32,8 +33,8 @@
                 <scan>
                     <horizontal>
-                        <samples>360</samples>
+                        <samples>90</samples>
                         <resolution>1</resolution>
-                        <min_angle>-3.14</min_angle>
-                        <max_angle>3.14</max_angle>
+                        <min_angle>0</min_angle>
+                        <max_angle>0.01</max_angle>
                     </horizontal>
                 </scan>

Commit message: lidar implemented, unable to rotate it

File: car_ros/description/robot_core.xacro (robot description, xacro)
@@ -190,36 +190,3 @@
         <material>Gazebo/Red</material>
     </gazebo>
-    <!-- ROTATING LINK -->
-    <joint name="rotate_joint" type="revolute">
-        <parent link="base_link"/>
-        <child link="rotate_link"/>
-        <origin xyz="-0.02 0 0.225" rpy="0 0 0"/>
-        <axis xyz="0 0 -1"/>
-        <limit lower="0" upper="${pi}" velocity="100" effort="100"/>
-    </joint>
-    <link name="rotate_link">
-        <visual>
-            <origin xyz="0 0 0" rpy="0 0 0"/>
-            <geometry>
-                <cylinder length="0.025" radius="0.025" />
-            </geometry>
-            <material name="orange" />
-        </visual>
-        <collision>
-            <origin xyz="0 0 0" rpy="-3.14159 0 0"/>
-            <geometry>
-                <cylinder length="0.001" radius="0.025" />
-            </geometry>
-        </collision>
-        <xacro:inertial_cylinder mass="0.01" length="0.001" radius="0.025">
-            <origin xyz="0 0 0" rpy="0 0 0"/>
-        </xacro:inertial_cylinder>
-    </link>
-    <gazebo>
-        <plugin name="gazebo_ros_joint_state_publisher"
-            filename="libgazebo_ros_joint_state_publisher.so">
-            <update_rate>40</update_rate>
-            <joint_name>rotate_link</joint_name>
-        </plugin>
-    </gazebo>
 </robot>

File: car_ros/description/robot_lidar.xacro (robot description, xacro)
@@ -2,6 +2,6 @@
 <robot xmlns:xacro="http://www.ros.org/wiki/xacro">
     <joint name="laser_joint" type="fixed">
-        <origin xyz = "0 0 0.025" rpy="0 0 0"/>
-        <parent link="rotate_link"/>
+        <origin xyz = "-0.02 0 0.1143" rpy="0 0 0"/>
+        <parent link="base_link"/>
         <child link="laser_frame"/>
     </joint>
@@ -34,12 +34,12 @@
                     <horizontal>
                         <samples>90</samples>
-                        <resolution>1</resolution>
-                        <min_angle>0</min_angle>
-                        <max_angle>0.01</max_angle>
+                        <resolution>10</resolution>
+                        <min_angle>-1.5708</min_angle>
+                        <max_angle>1.5708</max_angle>
                     </horizontal>
                 </scan>
                 <range>
                     <min>0.3</min>
-                    <max>12</max>
+                    <max>5</max>
                     <resolution>0.01</resolution>
                 </range>
